Commit message: 1.use last PND mpc controller 2.update adam_lite_simple and DuckDuck model files

File: Control/Sources/urdf/DuckDuck.urdf (robot description, URDF)
Before this commit: robot DuckDuck, 14 links, 13 joints
Links:
- removed link neck_pitch1
- removed link neck_pitch2
- added link left_ankle_roll, mass 0.0282743338823081; collision mesh filename=../meshes/left_ankle_roll.STL; visual mesh filename=../meshes/left_ankle_roll.STL
- added link neck_pitch, mass 0.0944141515929346; collision mesh filename=../meshes/neck_pitch.STL; visual mesh filename=../meshes/neck_pitch.STL
- added link neck_roll, mass 0.0554895568861581; collision mesh filename=../meshes/neck_roll.STL; visual mesh filename=../meshes/neck_roll.STL
- added link neck_yaw, mass 1.36489294645362; collision mesh filename=../meshes/neck_yaw.STL; visual mesh filename=../meshes/neck_yaw.STL
- added link right_ankle_roll, mass 0.0282743338823081; collision mesh filename=../meshes/right_ankle_roll.STL; visual mesh filename=../meshes/right_ankle_roll.STL
- link left_ankle_pitch: mass 0.0934205516990419 -> 0.0651489641090865
- link right_ankle_pitch: mass 0.0934206054212803 -> 0.0651490178313245
- link right_knee_pitch: mass 0.232718078417979 -> 0.232718078417978
Joints:
- removed joint neck_pitch1_joint
- removed joint neck_pitch2_joint
- added joint left_ankle_roll_joint: type revolute, parent left_ankle_pitch, child left_ankle_roll, origin xyz=0 0 -0.0523924267994756 rpy=0 0 0, axis 1 0 0, limit lower=0 upper=0 effort=0 velocity=0
- added joint neck_pitch_joint: type revolute, parent base, child neck_pitch, origin xyz=0.0774999999999999 0 0.108874586088177 rpy=0 0 0, axis 0 1 0, limit lower=0 upper=0 effort=0 velocity=0
- added joint neck_roll_joint: type revolute, parent neck_pitch, child neck_roll, origin xyz=0 -0.00249999999999992 0.0774999999999998 rpy=0 0 0, axis -1 0 0, limit lower=0 upper=0 effort=0 velocity=0
- added joint neck_yaw_joint: type revolute, parent neck_roll, child neck_yaw, origin xyz=0 0 0.061 rpy=0 0 0, axis 0 0 1, limit lower=0 upper=0 effort=0 velocity=0
- added joint right_ankle_roll_joint: type revolute, parent right_ankle_pitch, child right_ankle_roll, origin xyz=0 0 -0.0523924267994828 rpy=0 0 0, axis 1 0 0, limit lower=0 upper=0 effort=0 velocity=0

Commit message: Change joints positive direction for DuckDuck right leg
The DuckDuck zero statue is ok and add control for head

set rosopen is TRUE and compile for ros

File: Control/Sources/urdf/DuckDuck.urdf (robot description, URDF)
Before this commit: robot DuckDuck, 17 links, 16 joints
Joints:
- joint right_ankle_pitch_joint: axis 0 -1 0 -> 0 1 0
- joint right_ankle_roll_joint: axis 1 0 0 -> -1 0 0
- joint right_hip_pitch_joint: axis 0 -1 0 -> 0 1 0
- joint right_hip_roll_joint: axis 1 0 0 -> -1 0 0
- joint right_hip_yaw_joint: axis 0 0 1 -> 0 0 -1
- joint right_knee_pitch_joint: axis 0 -1 0 -> 0 1 0

Commit message: Z2S state not ok, still need to fix problem of wrong order for urdfreader
fix limit and boundingObject for DuckDuck.urdf and DuckDuck.wbt

add Z2S state bug recode

add test for zero state position jacobi in read_urdf.cpp

fix JointState_left_leg_v.xml

add Z2S and stand in state.cpp, but not test stand

File: Control/Sources/urdf/DuckDuck.urdf (robot description, URDF)
Before this commit: robot DuckDuck, 17 links, 16 joints
Joints:
- joint left_ankle_pitch_joint: limit lower=0 upper=0 effort=0 velocity=0 -> lower=-2 upper=2 effort=20 velocity=15.0
- joint left_ankle_roll_joint: limit lower=0 upper=0 effort=0 velocity=0 -> lower=-2 upper=2 effort=20 velocity=15.0
- joint left_hip_pitch_joint: limit lower=0 upper=0 effort=0 velocity=0 -> lower=-2 upper=2 effort=20 velocity=15.0
- joint left_hip_roll_joint: limit lower=0 upper=0 effort=0 velocity=0 -> lower=-2 upper=2 effort=20 velocity=15.0
- joint left_hip_yaw_joint: limit lower=0 upper=0 effort=0 velocity=0 -> lower=-2 upper=2 effort=20 velocity=15.0
- joint left_knee_pitch_joint: limit lower=0 upper=0 effort=0 velocity=0 -> lower=-2 upper=2 effort=20 velocity=15.0
- joint neck_pitch_joint: limit lower=0 upper=0 effort=0 velocity=0 -> lower=-2 upper=2 effort=20 velocity=15.0
- joint neck_roll_joint: limit lower=0 upper=0 effort=0 velocity=0 -> lower=-2 upper=2 effort=20 velocity=15.0
- joint neck_yaw_joint: limit lower=0 upper=0 effort=0 velocity=0 -> lower=-2 upper=2 effort=20 velocity=15.0
- joint right_ankle_pitch_joint: limit lower=0 upper=0 effort=0 velocity=0 -> lower=-2 upper=2 effort=20 velocity=15.0
- joint right_ankle_roll_joint: limit lower=0 upper=0 effort=0 velocity=0 -> lower=-2 upper=2 effort=20 velocity=15.0
- joint right_hip_pitch_joint: limit lower=0 upper=0 effort=0 velocity=0 -> lower=-2 upper=2 effort=20 velocity=15.0
- joint right_hip_roll_joint: limit lower=0 upper=0 effort=0 velocity=0 -> lower=-2 upper=2 effort=20 velocity=15.0
- joint right_hip_yaw_joint: limit lower=0 upper=0 effort=0 velocity=0 -> lower=-2 upper=2 effort=20 velocity=15.0
- joint right_knee_pitch_joint: limit lower=0 upper=0 effort=0 velocity=0 -> lower=-2 upper=2 effort=20 velocity=15.0

Commit message: fix problem of wrong joint order use tool of urdfreader read urdf files
check jacobi matrix and pose right

fix dataPub joint_name

change paras for joint PD and about wbc process

File: Control/Sources/urdf/DuckDuck.urdf (robot description, URDF)
Before this commit: robot DuckDuck, 17 links, 16 joints
Links:
- removed link neck_pitch
- removed link neck_roll
- removed link neck_yaw
- added link throat_pitch, mass 0.0944141515929346; collision mesh filename=../meshes/throat_pitch.STL; visual mesh filename=../meshes/throat_pitch.STL
- added link throat_roll, mass 0.0554895568861581; collision mesh filename=../meshes/throat_roll.STL; visual mesh filename=../meshes/throat_roll.STL
- added link throat_yaw, mass 1.36489294645362; collision mesh filename=../meshes/throat_yaw.STL; visual mesh filename=../meshes/throat_yaw.STL
Joints:
- removed joint neck_pitch_joint
- removed joint neck_roll_joint
- removed joint neck_yaw_joint
- added joint throat_pitch_joint: type revolute, parent base, child throat_pitch, origin xyz=0.0774999999999999 0 0.108874586088177 rpy=0 0 0, axis 0 1 0, limit lower=-2 upper=2 effort=20 velocity=15.0
- added joint throat_roll_joint: type revolute, parent throat_pitch, child throat_roll, origin xyz=0 -0.00249999999999992 0.0774999999999998 rpy=0 0 0, axis -1 0 0, limit lower=-2 upper=2 effort=20 velocity=15.0
- added joint throat_yaw_joint: type revolute, parent throat_roll, child throat_yaw, origin xyz=0 0 0.061 rpy=0 0 0, axis 0 0 1, limit lower=-2 upper=2 effort=20 velocity=15.0
